File: DAC_module.kicad_sch (KiCad schematic)
At the start: 20 parts, among them J2 Conn_01x05_Pin, J3 Conn_01x05_Pin, J5 Conn_02x04_Counter_Clockwise, U2 DAC80504

Commit message: Adding files of PCB v0.2
Parts:
- removed J5: Conn_02x04_Counter_Clockwise, Connector_PinHeader_2.54mm:PinHeader_2x04_P2.54mm_Vertical, symbol Connector_Generic:Conn_02x04_Counter_Clockwise
- added J1: Conn_01x06_Pin, Connector_PinHeader_2.54mm:PinHeader_1x06_P2.54mm_Vertical, symbol Connector:Conn_01x06_Pin
- J2: value Conn_01x05_Pin -> Conn_01x06_Pin; footprint Connector_PinHeader_2.54mm:PinHeader_1x05_P2.54mm_Vertical -> Connector_PinHeader_2.54mm:PinHeader_1x06_P2.54mm_Vertical; symbol Connector:Conn_01x05_Pin -> Connector:Conn_01x06_Pin
- J3: symbol Connector:Conn_01x05_Pin -> Connector:Conn_01x06_Pin
Connections:
- net CS: now also J2.4 (Pin_4); no longer J2.5 (Pin_5)
- net GND: now also J2.6 (Pin_6), J1.1 (Pin_1), J1.6 (Pin_6); no longer U2.3 (OUT1), U2.4 (OUT2), U2.5 (OUT3)
- net MISO: now also J2.5 (Pin_5); no longer J2.2 (Pin_2)
- net OUT0: now also J1.2 (Pin_2)
- net SCLK: now also J2.2 (Pin_2); no longer J2.4 (Pin_4)
- new net OUT1: J1.3 (Pin_3), U2.3 (OUT1)
- new net OUT2: J1.4 (Pin_4), U2.4 (OUT2)
- new net OUT3: J1.5 (Pin_5), U2.5 (OUT3)
